File: doc/schematics/Power Supply/PTN78000.sch (EAGLE design)
At the start: 5 parts, among them U1 1.5APOWERMODULE

Commit message: Schematics fixed
Parts:
- removed C4: (no value), rcl:C-EUC1206
- removed C5: (no value), rcl:CPOL-EUE5-6
- removed U1: 1.5APOWERMODULE, TIPOWERMODULE:1.5APOWERMODULE
- removed X: OUTPUT (6 V), con-wago-500:W237-102
- added C1: 2.2 uF, ASL:CAP1206
- added C2: 100 uF, ASL:CAP1206
- added JP1: M03PTH, ASL:M03PTH
- added U$1: PTN78000THROUGH-HOLE, ASL:PTN78000THROUGH-HOLE
- R1: value 13.1 K -> 21 K; device rcl:R-US_0207/10 -> ASL:RESISTOR1206
Connections:
- removed net VCC: U1.P$2
- new net N$3: C2.1, U$1.V_OUT
- new net N$4: JP1.3, U$1.INHIBIT
- net GND: now also C1.2, C2.2, JP1.2, R1.2, U$1.GND; no longer C4.2, C5.-, R1.1, U1.P$1
- net N$1: now also C1.1, JP1.1, U$1.V_IN; no longer R1.2, U1.P$4
- net N$2: now also R1.1, U$1.ADJ; no longer C4.1, C5.+, U1.P$5, X-2.KL
Other:
- moved on the sheet: R1

Commit message: New schematics
Parts:
- added F1: FUSE, ASL:FUSE
- added J11, J13, J14, J15, J16, J9: POW_CONNECTFEMALE-RA, ASL:POW_CONNECTFEMALE-RA
- added LED1: (no value), SparkFun-LED:LED5MM
- added R2: 330, ASL:RESISTOR1206
Connections:
- removed net N$3: C2.1, U$1.V_OUT
- new net N$5: C2.1, F1.1, F1.2, U$1.V_OUT
- new net N$6: LED1.A, R2.2
- new net VCC5V0: F1.3, F1.4, J11.1, J13.1, J14.1, J15.1, J16.1, J9.1, R2.1
- net GND: now also J11.2, J13.2, J14.2, J15.2, J16.2, J9.2, LED1.C
Changed lines of the file:
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@@
 <part name="GND1" library="ASL" deviceset="GND" device=""/>
 <part name="GND2" library="ASL" deviceset="GND" device=""/>
+<part name="J9" library="ASL" deviceset="POW_CONNECT" device="FEMALE-RA"/>
+<part name="U$2" library="ASL" deviceset="VCC5V0" device="" value="Output"/>
+<part name="U$3" library="ASL" deviceset="VCC5V0" device="" value="Output"/>
+<part name="GND4" library="ASL" deviceset="GND" device=""/>
+<part name="J11" library="ASL" deviceset="POW_CONNECT" device="FEMALE-RA"/>
+<part name="U$5" library="ASL" deviceset="VCC5V0" device="" value="Output"/>
+<part name="GND6" library="ASL" deviceset="GND" device=""/>
+<part name="J13" library="ASL" deviceset="POW_CONNECT" device="FEMALE-RA"/>
+<part name="U$7" library="ASL" deviceset="VCC5V0" device="" value="Output"/>
+<part name="GND8" library="ASL" deviceset="GND" device=""/>
+<part name="J14" library="ASL" deviceset="POW_CONNECT" device="FEMALE-RA"/>
+<part name="U$8" library="ASL" deviceset="VCC5V0" device="" value="Output"/>
+<part name="GND9" library="ASL" deviceset="GND" device=""/>
+<part name="J15" library="ASL" deviceset="POW_CONNECT" device="FEMALE-RA"/>
+<part name="U$9" library="ASL" deviceset="VCC5V0" device="" value="Output"/>
+<part name="GND10" library="ASL" deviceset="GND" device=""/>
+<part name="J16" library="ASL" deviceset="POW_CONNECT" device="FEMALE-RA"/>
+<part name="U$10" library="ASL" deviceset="VCC5V0" device="" value="Output"/>
+<part name="GND11" library="ASL" deviceset="GND" device=""/>
+<part name="F1" library="ASL" deviceset="FUSE" device=""/>
+<part name="R2" library="ASL" deviceset="RESISTOR" device="1206" value="330"/>
+<part name="U$4" library="ASL" deviceset="VCC5V0" device="" value="Output"/>
+<part name="LED1" library="SparkFun-LED" deviceset="LED" device="5MM"/>
+<part name="GND5" library="ASL" deviceset="GND" device=""/>
 </parts>
 <sheets>
@@
 <instance part="GND1" gate="1" x="22.86" y="167.64"/>
 <instance part="GND2" gate="1" x="91.44" y="167.64"/>
+<instance part="J9" gate="G$1" x="55.88" y="142.24"/>
+<instance part="U$2" gate="G$1" x="139.7" y="177.8"/>
+<instance part="U$3" gate="G$1" x="66.04" y="147.32"/>
+<instance part="GND4" gate="1" x="66.04" y="142.24"/>
+<instance part="J11" gate="G$1" x="55.88" y="111.76"/>
+<instance part="U$5" gate="G$1" x="66.04" y="116.84"/>
+<instance part="GND6" gate="1" x="66.04" y="111.76"/>
+<instance part="J13" gate="G$1" x="35.56" y="142.24"/>
+<instance part="U$7" gate="G$1" x="45.72" y="147.32"/>
+<instance part="GND8" gate="1" x="45.72" y="142.24"/>
+<instance part="J14" gate="G$1" x="35.56" y="127"/>
+<instance part="U$8" gate="G$1" x="45.72" y="132.08"/>
+<instance part="GND9" gate="1" x="45.72" y="127"/>
+<instance part="J15" gate="G$1" x="35.56" y="111.76"/>
+<instance part="U$9" gate="G$1" x="45.72" y="116.84"/>
+<instance part="GND10" gate="1" x="45.72" y="111.76"/>
+<instance part="J16" gate="G$1" x="35.56" y="96.52"/>
+<instance part="U$10" gate="G$1" x="45.72" y="101.6"/>
+<instance part="GND11" gate="1" x="45.72" y="96.52"/>
+<instance part="F1" gate="G$1" x="111.76" y="177.8"/>
+<instance part="R2" gate="G$1" x="99.06" y="139.7"/>
+<instance part="U$4" gate="G$1" x="93.98" y="139.7"/>
+<instance part="LED1" gate="G$1" x="106.68" y="137.16"/>
+<instance part="GND5" gate="1" x="106.68" y="129.54"/>
 </instances>
 <busses>
@@
 <pinref part="GND2" gate="1" pin="GND"/>
 </segment>
+<segment>
+<pinref part="J9" gate="G$1" pin="2"/>
+<pinref part="GND4" gate="1" pin="GND"/>
+</segment>
+<segment>
+<pinref part="J11" gate="G$1" pin="2"/>
+<pinref part="GND6" gate="1" pin="GND"/>
+</segment>
+<segment>
+<pinref part="J13" gate="G$1" pin="2"/>
+<pinref part="GND8" gate="1" pin="GND"/>
+</segment>
+<segment>
+<pinref part="J14" gate="G$1" pin="2"/>
+<pinref part="GND9" gate="1" pin="GND"/>
+</segment>
+<segment>
+<pinref part="J15" gate="G$1" pin="2"/>
+<pinref part="GND10" gate="1" pin="GND"/>
+</segment>
+<segment>
+<pinref part="J16" gate="G$1" pin="2"/>
+<pinref part="GND11" gate="1" pin="GND"/>
+</segment>
+<segment>
+<pinref part="LED1" gate="G$1" pin="C"/>
+<pinref part="GND5" gate="1" pin="GND"/>
+</segment>
 </net>
 <net name="N$2" class="0">
@@
 <pinref part="U$1" gate="G$1" pin="ADJ"/>
 <pinref part="R1" gate="G$1" pin="1"/>
-</segment>
-</net>
-<net name="N$3" class="0">
-<segment>
-<pinref part="U$1" gate="G$1" pin="V_OUT"/>
-<wire x1="71.12" y1="177.8" x2="91.44" y2="177.8" width="0.2032" layer="91"/>
-<wire x1="91.44" y1="177.8" x2="109.22" y2="177.8" width="0.2032" layer="91"/>
-<wire x1="109.22" y1="177.8" x2="109.22" y2="175.26" width="0.2032" layer="91"/>
-<wire x1="109.22" y1="175.26" x2="119.38" y2="175.26" width="0.2032" layer="91"/>
-<pinref part="C2" gate="G$1" pin="1"/>
-<junction x="91.44" y="177.8"/>
 </segment>
 </net>
@@
 </segment>
 </net>
+<net name="VCC5V0" class="0">
+<segment>
+<pinref part="J9" gate="G$1" pin="1"/>
+<pinref part="U$3" gate="G$1" pin="VCC5V0"/>
+</segment>
+<segment>
+<pinref part="J11" gate="G$1" pin="1"/>
+<pinref part="U$5" gate="G$1" pin="VCC5V0"/>
+</segment>
+<segment>
+<pinref part="J13" gate="G$1" pin="1"/>
+<pinref part="U$7" gate="G$1" pin="VCC5V0"/>
+</segment>
+<segment>
+<pinref part="J14" gate="G$1" pin="1"/>
+<pinref part="U$8" gate="G$1" pin="VCC5V0"/>
+</segment>
+<segment>
+<pinref part="J15" gate="G$1" pin="1"/>
+<pinref part="U$9" gate="G$1" pin="VCC5V0"/>
+</segment>
+<segment>
+<pinref part="J16" gate="G$1" pin="1"/>
+<pinref part="U$10" gate="G$1" pin="VCC5V0"/>
+</segment>
+<segment>
+<pinref part="U$2" gate="G$1" pin="VCC5V0"/>
+<pinref part="F1" gate="G$1" pin="3"/>
+<wire x1="139.7" y1="177.8" x2="121.92" y2="177.8" width="0.2032" layer="91"/>
+<pinref part="F1" gate="G$1" pin="4"/>
+<wire x1="121.92" y1="177.8" x2="121.92" y2="175.26" width="0.2032" layer="91"/>
+</segment>
+<segment>
+<pinref part="R2" gate="G$1" pin="1"/>
+<pinref part="U$4" gate="G$1" pin="VCC5V0"/>
+</segment>
+</net>
+<net name="N$5" class="0">
+<segment>
+<pinref part="U$1" gate="G$1" pin="V_OUT"/>
+<wire x1="71.12" y1="177.8" x2="91.44" y2="177.8" width="0.2032" layer="91"/>
+<pinref part="C2" gate="G$1" pin="1"/>
+<pinref part="F1" gate="G$1" pin="1"/>
+<pinref part="F1" gate="G$1" pin="2"/>
+<wire x1="91.44" y1="177.8" x2="101.6" y2="177.8" width="0.2032" layer="91"/>
+<wire x1="101.6" y1="177.8" x2="101.6" y2="180.34" width="0.2032" layer="91"/>
+</segment>
+</net>
+<net name="N$6" class="0">
+<segment>
+<pinref part="R2" gate="G$1" pin="2"/>
+<pinref part="LED1" gate="G$1" pin="A"/>
+<wire x1="106.68" y1="139.7" x2="104.14" y2="139.7" width="0.1524" layer="91"/>
+</segment>
+</net>
