File: doc/schematics/IO shields/AtLAs/IO Shield_With_Power_Supply_PCB.brd (EAGLE design)
At the start: 76.2 x 83.8 mm, 40 parts, among them IC1 74S08D, IC2 74LS04D, IC3 74S08D, IC4 74LS32D, J1 POW_CONNECTFEMALE-RA

Commit message: Merged in Johns physical design changes.
Parts:
- removed C10: 0.1uf, resistor:C0805
- removed INTERNAL_POWER: FUSE, ASL:FUSE_2AG
- removed JP14: (no value), pinhead:1X06
- removed JP16: (no value), pinhead:2X08
- added C5: 0.1uf, resistor:C0805
- added C6: 47uf, resistor:C0805
- added J4, J5: POW_CONNECTFEMALE-RA, ASL:SOCKET-FEMALE_RA-3.96MM-2
- added JP10, JP12: (no value), pinhead:1X04/90
- added LED1, LED10, LED11, LED2, LED3, LED5, LED6, LED7, LED9: (no value), ASL:FKIT-LED-1206
- added R10, R11, R3, R4, R5, R6, R7, R8, R9: 470, ASL:0805
- added R2: 4.7K, ASL:0805
- added U$6: PTN78000, ASL:PTN78000
- added U$7: LM3940IMP-3.3, LM3940:SOT223
- added XB1: XBEE-PRO, maxstream:XBEE-PRO
- C3: value 47uf -> 0.1uf
- JP11: device pinhead:2X08 -> pinhead:1X04/90
- JP13: device pinhead:2X06 -> baro:1X06
- moved JP11 80.0 mm to (81.3, 26.0), flipped to the bottom, turned to 90 degrees
- moved J1 63.5 mm to (11.4, 53.3), turned to 270 degrees
- moved JP8 61.6 mm to (20.3, 63.5), turned to 180 degrees
- moved U$1 40.6 mm to (73.7, 62.2), turned to 90 degrees
- moved C2 38.9 mm to (74.3, 67.9)
- moved JP17 38.6 mm to (66.0, 26.7), turned to 270 degrees
- moved C4 30.2 mm to (62.2, 24.1), turned to 270 degrees
- moved C1 28.6 mm to (78.1, 57.8), turned to 180 degrees
- moved C3 25.5 mm to (66.0, 14.0)
- moved JP13 24.3 mm to (57.1, 52.1), turned to 180 degrees
- moved EXTERNAL_POWER 20.9 mm to (77.5, 48.3), turned to 0 degrees
- moved D1 7.96 mm to (71.8, 48.3)
- moved JP1 2.84 mm to (39.4, -2.54)
- moved JP2 2.84 mm to (48.3, -2.54)
- moved JP3 2.84 mm to (57.1, -2.54)
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Connections:
- removed net N$11: C1.2, D1.C, EXTERNAL_POWER.P$3, EXTERNAL_POWER.P$4, JP14.1, JP7.1, U$1.1
- removed net N$27 (its old number): JP11.8, JP4.8
- removed net N$29: JP11.12, JP4.12
- removed net N$30: JP11.10, JP4.10
- removed net N$31: JP13.3, JP6.3
- removed net N$32: JP15.3, JP16.3
- removed net N$33: JP15.5, JP16.5
- removed net N$34: JP15.7, JP16.7
- removed net N$36: JP15.13, JP16.13
- removed net N$37: JP15.11, JP16.11
- removed net N$38: JP15.9, JP16.9
- removed net N$39: JP15.2, JP16.2
- removed net N$40: JP15.4, JP16.4
- removed net N$41: JP13.5, JP6.5
- removed net N$42: JP15.8, JP16.8
- removed net N$44: INTERNAL_POWER.P$1, INTERNAL_POWER.P$2, JP14.4, JP7.4
- removed net N$45: JP15.10, JP16.10
- removed net N$46: JP13.7, JP6.7
- removed net N$47: JP13.9, JP6.9
- removed net N$48: JP13.11, JP6.11
- removed net N$49: JP13.2, JP5.4, JP6.2
- removed net N$50: JP13.4, JP5.3, JP6.4
- removed net N$51: JP13.6, JP6.6
- removed net N$52: JP13.8, JP6.8
- removed net N$53: JP13.10, JP6.10
- removed net N$58: JP14.5, JP7.5
- removed net N$59: JP14.6, JP7.6
- removed net REC_ENABLE: JP15.16, JP16.16
- new net N$35: R2.2, U$6.ADJ
- new net N$7: JP12.2, JP15.8
- new net SCL: JP10.1, JP13.2, JP5.4, JP6.2
- new net SDA: JP10.2, JP13.1, JP5.3, JP6.4, LED10.A
- new net XBEE_RX: JP4.1, JP9.4, LED11.A, XB1.2
- new net XBEE_TX: JP4.3, JP9.5, LED3.A, XB1.3
- net ENABLE: no longer JP16.6
- net GND: now also C3.1, C5.1, C6.2, J4.2, J5.2, JP10.4, JP11.4, JP12.4, JP13.5, R10.1, R11.1, R2.1, R3.1, R4.1, R5.1, R6.1, R7.1, R8.1, R9.1, U$6.GND, U$7.2, XB1.10; no longer C10.2, C3.2, JP14.2, JP14.3
- net GPS_RX: now also JP11.3, JP15.12, JP17.2, LED9.A; no longer JP15.14, JP16.14, JP17.3
- net GPS_TX: now also JP11.2, JP15.14, JP17.3; no longer JP15.12, JP16.12, JP17.2
- net L.MOTOR: no longer JP16.1
- net N$10: now also LED7.A
- net N$13: now also U$6.V_IN; no longer C10.1, C3.1, J1.1
- net N$14: no longer JP16.15
- net N$15: now also C5.2, U$7.3, XB1.1; no longer JP13.1, JP6.1
- net N$17: now also LED3.C, R11.2; no longer JP11.3, JP4.3, JP9.5
- net N$18: no longer JP11.5
- net N$19: now also LED10.C, R3.2; no longer JP11.7, JP4.7
- net N$20: now also LED11.C, R4.2; no longer JP11.15, JP4.15
- net N$21: now also LED9.C, R5.2; no longer JP11.13, JP4.13
- net N$22: now also LED5.C, R6.2; no longer JP11.11, JP4.11
- net N$23: now also LED6.C, R7.2; no longer JP11.9, JP4.9
- net N$24: now also LED7.C, R8.2; no longer JP11.2, JP4.2
- net N$25: now also LED1.C, R9.2; no longer JP11.4, JP4.4
- net N$26: now also LED2.C, R10.2; no longer JP11.6, JP4.6
- net N$28: now also EXTERNAL_POWER.P$3, EXTERNAL_POWER.P$4, J5.1; no longer JP11.14, JP4.14
- net N$4: now also JP12.1, JP6.10; no longer JP11.1, JP4.1, JP9.4
- net N$8: now also LED5.A
- net N$9: now also LED6.A
- net R.MOTOR: no longer JP11.16
- net RUDDER: no longer JP13.12
- net VCC: now also C1.2, C3.2, C6.1, D1.C, J1.1, J4.1, JP10.3, JP11.1, JP12.3, JP13.6, JP7.1, LED1.A, U$1.1, U$6.V_OUT, U$7.1; no longer INTERNAL_POWER.P$3, INTERNAL_POWER.P$4
- net VDD: now also LED2.A
Routing:
- net VCC: track 29.7 -> 221.8 mm, vias 4 -> 10
- net N$11: track 91.1 -> 0.00 mm
- net XBEE_TX: track 0.00 -> 83.9 mm
- net XBEE_RX: track 0.00 -> 79.3 mm
- net N$12: track 30.6 -> 104.6 mm, vias 0 -> 2
- net SCL: track 0.00 -> 49.7 mm
- net SDA: track 0.00 -> 49.2 mm
- net N$4: track 27.1 -> 75.0 mm
- net N$7: track 0.00 -> 40.0 mm
- net N$13: track 21.3 -> 60.7 mm
- net VDD: track 64.8 -> 28.6 mm, vias 2 -> 1
- net N$17: track 23.5 -> 1.49 mm
- net GPS_RX: track 44.6 -> 64.8 mm, vias 0 -> 1
- net N$50: track 18.1 -> 0.00 mm
- net N$49: track 18.1 -> 0.00 mm
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Other:
- board size 76.2 x 83.8 mm -> 78.7 x 83.8 mm
