File: doc/schematics/IO shields/AtLAs/IO Shield_With_Power_Supply_PCB.sch (EAGLE design)
At the start: 58 parts, among them IC1 74S08D, IC2 74LS04D, IC3 74S08D, IC4 74LS32D, J1 POW_CONNECTFEMALE-RA, J4 POW_CONNECTFEMALE-RA, J5 POW_CONNECTFEMALE-RA

Commit message: Merged in Johns physical design changes.
Parts:
- removed INTERNAL_POWER: FUSE, ASL:FUSE
- added JP13: (no value), baro:PINHD-1X6
- added LED3: (no value), ASL:LED-FKIT-1206
- added R11: 470, ASL:RESISTOR0805-RES
- U$6: value PTN78000THROUGH-HOLE -> PTN78000
Connections:
- net N$4 renamed XBEE_RX
- removed net N$11: C1.2, D1.C, EXTERNAL_POWER.3, EXTERNAL_POWER.4, JP7.1, U$1.IN
- removed net N$16: J5.1, LED1.A, U$6.V_IN
- removed net N$43: C3.1, R2.1
- removed net N$44: INTERNAL_POWER.1, INTERNAL_POWER.2, JP7.4
- removed net N$49: JP10.1, JP5.4, JP6.2
- removed net N$50: JP10.2, JP5.3, JP6.4, LED10.A
- new net N$28: EXTERNAL_POWER.3, EXTERNAL_POWER.4, J5.1
- new net N$4: JP12.1, JP6.10
- new net N$7: JP12.2, JP15.8
- new net SCL: JP10.1, JP13.2, JP5.4, JP6.2
- new net SDA: JP10.2, JP13.1, JP5.3, JP6.4, LED10.A
- new net XBEE_TX: JP4.3, JP9.5, LED3.A, XB1.DIN/!CONFIG
- net GND: now also C3.1, JP13.5, R11.1, R2.1
- net GPS_RX: now also JP11.3, JP15.12, JP17.2, LED9.A; no longer JP11.2, JP15.14, JP17.3
- net GPS_TX: now also JP11.2, JP15.14, JP17.3; no longer JP11.3, JP15.12, JP17.2, LED9.A
- net N$13: now also U$6.V_IN; no longer C3.2, U$6.V_OUT
- net N$17: now also LED3.C, R11.2; no longer JP4.3, JP9.5, XB1.DIN/!CONFIG
- net VCC: now also C1.2, C3.2, D1.C, JP13.6, JP7.1, LED1.A, U$1.IN, U$6.V_OUT; no longer INTERNAL_POWER.3, INTERNAL_POWER.4
Other:
- moved on the sheet: D1, EXTERNAL_POWER, J5, LED1, LED11, R4, R9
