File: doc/schematics/IO shields/Command Center/IO Shield_With_Power_Supply_PCB.brd (EAGLE design)
At the start: 78.7 x 83.8 mm, 62 parts, among them IC1 74S08D, IC2 74LS04D, IC3 74S08D, IC4 74LS32D, J1 POW_CONNECTFEMALE-RA, J4 POW_CONNECTFEMALE-RA, J5 POW_CONNECTFEMALE-RA

Commit message: Merged in Johns physical design changes.
Parts:
- removed C11, C12, C13, C14, C8, C9: 0.1uf, resistor:C0805
- removed IC1, IC3: 74S08D, 74xx-us:SO14
- removed IC2: 74LS04D, 74xx-us:SO14
- removed IC4: 74LS32D, 74xx-us:SO14
- removed INTERNAL_POWER: FUSE, ASL:FUSE_2AG
- removed J4, J5: POW_CONNECTFEMALE-RA, ASL:SOCKET-FEMALE_RA-3.96MM-2
- removed JP10, JP11, JP12: (no value), pinhead:1X04/90
- removed JP5: (no value), SDLogger:1X04
- removed LED10, LED11, LED2, LED5, LED6, LED7, LED9: (no value), ASL:FKIT-LED-1206
- removed R1: 4.7K, ASL:0805
- removed R10, R3, R4, R5, R6, R7, R8: 470, ASL:0805
- removed U$1: LM3940IMP-3.3, LM3940:SOT223
- added C7: 0.1uf, resistor:C0805
- added SL1, SL2: (no value), ASL:1X04_LOCK
- C1, C6: value 47uf -> 0.1uf
- C2: value 0.1uf -> 4.7uf
- C3: value 0.1uf -> 100uF
- C5: value 0.1uf -> 2.2uF
- J1: value POW_CONNECTFEMALE-RA -> POW_CONNECTMALE; device ASL:SOCKET-FEMALE_RA-3.96MM-2 -> ASL:SOCKET-MALE-3.96MM-2
- JP1: device pinhead:1X03/90 -> pinhead_non_standard:1X04
- JP2: device pinhead:1X03/90 -> pinhead:1X04/90
- JP3: device pinhead:1X03/90 -> pinhead:1X02
- JP8: device pinhead:2X04 -> baro:1X06
- JP9: device SDLogger:1X06 -> pinhead:2X15/90
- moved JP3 89.8 mm to (14.0, 76.2), turned to 0 degrees
- moved JP1 76.2 mm to (39.4, 73.7), turned to 90 degrees
- moved C5 70.3 mm to (78.4, 41.6)
- moved C1 68.8 mm to (9.21, 29.2), turned to 180 degrees
- moved JP9 68.1 mm to (52.7, 0.00), flipped to the bottom
- moved C2 63.6 mm to (9.21, 39.4)
- moved J1 63.5 mm to (73.3, 67.3), turned to 180 degrees
- moved C6 58.2 mm to (59.7, 61.0), turned to 90 degrees
- moved R2 55.6 mm to (80.6, 63.8)
- moved JP2 51.3 mm to (82.5, 35.6), turned to 270 degrees
- moved U$6 41.9 mm to (71.1, 44.5)
- moved JP8 33.3 mm to (53.3, 67.9), turned to 0 degrees
- moved EXTERNAL_POWER 32.9 mm to (78.1, 17.8), turned to 180 degrees
- moved C3 13.7 mm to (69.2, 27.3)
- moved U$7 13.6 mm to (11.7, 34.3)
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Connections:
- removed net ENABLE: IC2.13, IC3.10, IC3.13, IC3.2, JP15.6, R1.2
- removed net L.MOTOR: IC3.9, JP15.1
- removed net N$14: JP15.15, JP8.10
- removed net N$43: C3.1, R2.1
- removed net N$44: INTERNAL_POWER.P$1, INTERNAL_POWER.P$2, JP7.4
- removed net N$49: JP10.1, JP5.4, JP6.2
- removed net N$50: JP10.2, JP5.3, JP6.4, LED10.A
- removed net R.MOTOR: IC3.12, JP4.16
- removed net REC.MOTOR: IC1.5, JP8.11
- removed net REC_RUDDER: IC1.1, JP8.12
- removed net RUDDER: IC3.1, JP6.12
- removed net VDD: C2.1, C8.1, JP5.2, LED2.A, U$1.3
- new net N$28: JP15.4, JP9.12
- new net N$31: JP15.3, JP9.20
- new net N$36: JP1.3, JP6.4, JP8.1, JP9.24, SL1.2, SL2.2
- new net N$7: JP15.2, JP9.4
- new net XBEE_RX: JP3.2, JP4.1
- new net XBEE_TX: JP4.3, XB1.3
- net GND: now also C2.1, C3.1, C5.2, C6.1, C7.1, J1.P$2, JP1.1, JP2.1, JP9.27, JP9.28, R2.1, SL1.4, SL2.4; no longer C11.1, C12.1, C13.1, C14.1, C2.2, C5.1, C6.2, C8.2, C9.2, IC1.10, IC1.12, IC1.13, IC1.7, IC1.9, IC2.1, IC2.11, IC2.3, IC2.5, IC2.7, IC2.9, IC3.4, IC3.5, IC3.7, IC4.12, IC4.13, IC4.7, J1.2, J4.2, J5.2, JP1.3, JP10.4, JP11.4, JP12.4, JP2.3, JP3.3, JP5.1, JP7.3, JP8.1, JP8.3, JP8.7, JP9.1, JP9.2, R1.1, R10.1, R3.1, R4.1, R5.1, R6.1, R7.1, R8.1, U$1.2
- net GPS_RX: now also JP17.2, JP2.2; no longer JP11.2, JP17.3
- net GPS_TX: now also JP17.3, JP2.3; no longer JP11.3, JP17.2, LED9.A
- net N$1: now also JP3.1, XB1.2; no longer IC1.3, IC4.1
- net N$10: now also JP4.12, JP9.9; no longer IC4.8, JP3.1, LED7.A
- net N$11: now also JP15.5, JP9.10; no longer C1.2, D1.C, EXTERNAL_POWER.P$3, EXTERNAL_POWER.P$4, JP7.1, U$1.1
- net N$12: now also JP4.10, JP9.11; no longer JP1.2, JP2.2, JP8.8
- net N$13: now also C1.2, C6.2, C7.2, JP1.2, JP8.6, SL1.3, SL2.3, U$7.3, XB1.1; no longer C3.2, EXTERNAL_POWER.P$1, EXTERNAL_POWER.P$2, U$6.V_OUT
- net N$15: now also JP4.8, JP9.13; no longer C5.2, U$7.3, XB1.1
- net N$16: now also C5.1, EXTERNAL_POWER.P$3, EXTERNAL_POWER.P$4; no longer J5.1, LED1.A
- net N$17: now also JP4.6, JP9.15; no longer JP4.3, JP9.5, XB1.3
- net N$18: now also JP4.4, JP9.17; no longer JP4.5, JP9.6
- net N$19: now also JP4.2, JP9.19; no longer LED10.C, R3.2
- net N$2: now also JP4.5, JP9.1; no longer IC1.6, IC4.4, IC4.9
- net N$20: now also JP4.15, JP9.21; no longer LED11.C, R4.2
- net N$21: now also JP4.13, JP9.23; no longer LED9.C, R5.2
- net N$22: now also JP4.11, JP9.25; no longer LED5.C, R6.2
- net N$23: now also JP15.8, JP9.14; no longer LED6.C, R7.2
- net N$24: now also JP15.6, JP9.18; no longer LED7.C, R8.2
- net N$26: now also JP1.4, JP6.2, JP8.2, JP9.22, SL1.1, SL2.1; no longer LED2.C, R10.2
- net N$27: now also JP15.10, JP9.16; no longer IC3.3, IC4.2
- net N$3: now also EXTERNAL_POWER.P$1, EXTERNAL_POWER.P$2, J1.P$1; no longer IC1.2, IC1.4, IC2.12
- net N$4: now also JP4.9, JP9.3; no longer JP4.1, JP9.4, LED11.A, XB1.2
- net N$5: now also JP4.7, JP9.6; no longer IC3.11, IC4.10
- net N$6: now also JP15.1, JP9.2; no longer IC3.8, IC4.5
- net N$8: now also JP4.16, JP9.5; no longer IC4.6, JP1.1, LED5.A
- net N$9: now also JP4.14, JP9.7; no longer IC4.3, JP2.1, LED6.A
- net VCC: now also C2.2, C3.2, D1.C, JP2.4, JP7.1, JP9.30, LED1.A, U$6.V_OUT; no longer C11.2, C12.2, C13.2, C14.2, C6.1, C9.1, IC1.14, IC2.14, IC3.14, IC4.14, INTERNAL_POWER.P$3, INTERNAL_POWER.P$4, J1.1, J4.1, JP10.3, JP11.1, JP12.3, JP9.3
Routing:
- net N$13: track 35.9 -> 177.5 mm, vias 0 -> 5
- net N$36: track 0.00 -> 133.4 mm, vias 0 -> 4
- net N$26: track 2.76 -> 123.9 mm, vias 0 -> 3
- net N$5: track 12.3 -> 97.0 mm, vias 0 -> 1
- net N$22: track 2.76 -> 85.8 mm, vias 0 -> 1
- net N$19: track 2.76 -> 84.8 mm
- net N$21: track 2.63 -> 81.9 mm, vias 0 -> 1
- net GPS_RX: track 62.5 -> 138.9 mm, vias 0 -> 5
- net N$31: track 0.00 -> 75.6 mm, vias 0 -> 1
- net N$20: track 2.76 -> 78.3 mm, vias 0 -> 1
- net GPS_TX: track 64.8 -> 139.9 mm, vias 1 -> 5
- net N$18: track 11.2 -> 81.3 mm
- net N$24: track 2.76 -> 66.9 mm, vias 0 -> 1
- net N$7: track 0.00 -> 60.5 mm
- net N$28: track 0.00 -> 60.3 mm, vias 0 -> 1
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- removed copper zone on layer 16, net VCC
Other:
- board size 78.7 x 83.8 mm -> 80 x 83.8 mm
